File: gpswide.sch (KiCad schematic (older format))
At the start: 12 parts, among them J1 GPS E406A, J2 Raspberry Pi, Q1 2N3904, U1 NE555

Commit message: cleaned up
Connections:
- net labels added: GPS_GND, GPS_PPS, GPS_TX, GPS_VCC, GPX_GND, RPI_GND, RPI_PPS, RPI_RX, RPI_VCC
- wire segments 63 -> 47
Changed lines of the file:
@@
 $EndComp
-Wire Wire Line
-	8200 2200 8200 1650
-Wire Wire Line
-	8200 2500 8200 3350
 Wire Wire Line
 	4200 1650 4200 2400
 Wire Wire Line
 	4200 2700 4200 3350
-Connection ~ 7800 2400
-Wire Wire Line
-	4500 2500 4500 1700
-Wire Wire Line
-	4500 1700 8000 1700
-Wire Wire Line
-	8000 1700 8000 2300
 $Comp
 L Connector:Conn_01x08_Male J1
 U 1 1 5B705252
-P 3450 2900
-F 0 "J1" H 3556 3378 50  0000 C CNN
-F 1 "GPS E406A" H 3556 3287 50  0000 C CNN
-F 2 "Connector_PinHeader_2.54mm:PinHeader_1x08_P2.54mm_Vertical" H 3450 2900 50  0001 C CNN
-F 3 "~" H 3450 2900 50  0001 C CNN
-	1    3450 2900
+P 4350 5200
+F 0 "J1" H 4456 5678 50  0000 C CNN
+F 1 "GPS E406A" H 4456 5587 50  0000 C CNN
+F 2 "Connector_PinHeader_2.54mm:PinHeader_1x08_P2.54mm_Vertical" H 4350 5200 50  0001 C CNN
+F 3 "~" H 4350 5200 50  0001 C CNN
+	1    4350 5200
 	1    0    0    -1
 $EndComp
-Wire Wire Line
-	3650 2600 4550 2600
-Wire Wire Line
-	4000 2500 4000 2800
-Wire Wire Line
-	4000 2800 3650 2800
-Wire Wire Line
-	4000 2500 4500 2500
-Wire Wire Line
-	4200 2400 3900 2400
-Wire Wire Line
-	3900 2400 3900 3000
-Wire Wire Line
-	3900 3000 3650 3000
-Wire Wire Line
-	4200 2700 4100 2700
-Wire Wire Line
-	4100 2700 4100 3100
-Wire Wire Line
-	4100 3100 3650 3100
 $Comp
 L Connector_Generic:Conn_02x08_Odd_Even J2
 U 1 1 5B7079DD
-P 9000 2500
-F 0 "J2" H 9050 3017 50  0000 C CNN
-F 1 "Raspberry Pi" H 9050 2926 50  0000 C CNN
-F 2 "Connector_PinSocket_2.54mm:PinSocket_2x08_P2.54mm_Vertical" H 9000 2500 50  0001 C CNN
-F 3 "~" H 9000 2500 50  0001 C CNN
-	1    9000 2500
+P 6850 5200
+F 0 "J2" H 6900 5717 50  0000 C CNN
+F 1 "Raspberry Pi" H 6900 5626 50  0000 C CNN
+F 2 "Connector_PinSocket_2.54mm:PinSocket_2x08_P2.54mm_Vertical" H 6850 5200 50  0001 C CNN
+F 3 "~" H 6850 5200 50  0001 C CNN
+	1    6850 5200
 	1    0    0    -1
 $EndComp
+Text GLabel 3950 2400 0    50   Output ~ 0
+GPS_VCC
+Text GLabel 3950 2700 0    50   Output ~ 0
+GPX_GND
+Text GLabel 3950 2600 0    50   Input ~ 0
+GPS_PPS
+Text GLabel 3950 2500 0    50   Input ~ 0
+GPS_TX
+Text GLabel 4700 5300 2    50   Output ~ 0
+GPS_VCC
+Text GLabel 4700 5400 2    50   Output ~ 0
+GPS_GND
+Text GLabel 4700 4900 2    50   Input ~ 0
+GPS_PPS
+Text GLabel 4700 5100 2    50   Input ~ 0
+GPS_TX
 Wire Wire Line
-	8200 2200 8350 2200
+	4550 4900 4700 4900
 Wire Wire Line
-	8350 2200 8350 1850
+	4550 5100 4700 5100
 Wire Wire Line
-	8350 1850 9550 1850
+	4550 5300 4700 5300
 Wire Wire Line
-	9550 1850 9550 2300
+	4200 2400 3950 2400
 Wire Wire Line
-	9550 2300 9300 2300
+	4550 2600 3950 2600
 Wire Wire Line
-	8200 2500 8550 2500
+	3950 2700 4200 2700
 Wire Wire Line
-	8550 2500 8550 3100
+	4550 5400 4700 5400
+Text GLabel 7350 5100 2    50   Input ~ 0
+RPI_GND
+Text GLabel 7350 5300 2    50   Output ~ 0
+RPI_RX
+Text GLabel 7350 5000 2    50   Input ~ 0
+RPI_VCC
+Text GLabel 6450 5200 0    50   Output ~ 0
+RPI_PPS
 Wire Wire Line
-	8550 3100 9550 3100
+	6450 5200 6650 5200
 Wire Wire Line
-	9550 3100 9550 2400
+	7150 5000 7350 5000
 Wire Wire Line
-	9550 2400 9300 2400
+	7150 5100 7350 5100
 Wire Wire Line
-	8550 2300 8550 1900
+	7150 5300 7350 5300
+Text GLabel 4200 2500 2    50   Input ~ 0
+RPI_RX
 Wire Wire Line
-	8550 1900 9650 1900
+	3950 2500 4200 2500
+Text GLabel 8450 1800 2    50   Output ~ 0
+RPI_VCC
+Text GLabel 8450 3200 2    50   Output ~ 0
+RPI_GND
+Text GLabel 8450 2400 2    50   Output ~ 0
+RPI_PPS
 Wire Wire Line
-	9650 1900 9650 2600
+	8450 1800 8200 1800
 Wire Wire Line
-	9650 2600 9300 2600
+	8200 1800 8200 1650
 Wire Wire Line
-	8000 2300 8550 2300
+	8450 3200 8200 3200
 Wire Wire Line
-	8700 2400 8700 2500
+	8200 3200 8200 3350
 Wire Wire Line
-	8700 2500 8800 2500
-Wire Wire Line
-	7800 2400 8700 2400
+	8450 2400 7800 2400
+Connection ~ 7800 2400
 $EndSCHEMATC

Commit message: ground plane added
Connections:
- net labels removed: GPS_GND, GPX_GND, RPI_GND
- wire segments 47 -> 45
Changed lines of the file:
@@
-$EndComp
-$Comp
-L power:GND #PWR0109
-U 1 1 5B7223D5
-P 8200 3350
-F 0 "#PWR0109" H 8200 3100 50  0001 C CNN
-F 1 "GND" H 8205 3177 50  0000 C CNN
-F 2 "" H 8200 3350 50  0001 C CNN
-F 3 "" H 8200 3350 50  0001 C CNN
-	1    8200 3350
-	1    0    0    -1
-$EndComp
-$Comp
-L power:GND #PWR0110
-U 1 1 5B72246F
-P 4200 3350
-F 0 "#PWR0110" H 4200 3100 50  0001 C CNN
-F 1 "GND" H 4205 3177 50  0000 C CNN
-F 2 "" H 4200 3350 50  0001 C CNN
-F 3 "" H 4200 3350 50  0001 C CNN
-	1    4200 3350
-	1    0    0    -1
 $EndComp
 $Comp
@@
 Wire Wire Line
 	4200 1650 4200 2400
-Wire Wire Line
-	4200 2700 4200 3350
 $Comp
 L Connector:Conn_01x08_Male J1
@@
 Text GLabel 3950 2400 0    50   Output ~ 0
 GPS_VCC
-Text GLabel 3950 2700 0    50   Output ~ 0
-GPX_GND
 Text GLabel 3950 2600 0    50   Input ~ 0
 GPS_PPS
@@
 Text GLabel 4700 5300 2    50   Output ~ 0
 GPS_VCC
-Text GLabel 4700 5400 2    50   Output ~ 0
-GPS_GND
 Text GLabel 4700 4900 2    50   Input ~ 0
 GPS_PPS
@@
 	4550 2600 3950 2600
 Wire Wire Line
-	3950 2700 4200 2700
-Wire Wire Line
 	4550 5400 4700 5400
-Text GLabel 7350 5100 2    50   Input ~ 0
-RPI_GND
 Text GLabel 7350 5300 2    50   Output ~ 0
 RPI_RX
@@
 	7150 5000 7350 5000
 Wire Wire Line
-	7150 5100 7350 5100
-Wire Wire Line
 	7150 5300 7350 5300
 Text GLabel 4200 2500 2    50   Input ~ 0
@@
 Text GLabel 8450 1800 2    50   Output ~ 0
 RPI_VCC
-Text GLabel 8450 3200 2    50   Output ~ 0
-RPI_GND
 Text GLabel 8450 2400 2    50   Output ~ 0
 RPI_PPS
@@
 	8200 1800 8200 1650
 Wire Wire Line
-	8450 3200 8200 3200
-Wire Wire Line
-	8200 3200 8200 3350
-Wire Wire Line
 	8450 2400 7800 2400
 Connection ~ 7800 2400
+$Comp
+L power:GND #PWR?
+U 1 1 5B71BD00
+P 4700 5950
+F 0 "#PWR?" H 4700 5700 50  0001 C CNN
+F 1 "GND" H 4705 5777 50  0000 C CNN
+F 2 "" H 4700 5950 50  0001 C CNN
+F 3 "" H 4700 5950 50  0001 C CNN
+	1    4700 5950
+	1    0    0    -1
+$EndComp
+$Comp
+L power:GND #PWR?
+U 1 1 5B71BD46
+P 7750 6000
+F 0 "#PWR?" H 7750 5750 50  0001 C CNN
+F 1 "GND" H 7755 5827 50  0000 C CNN
+F 2 "" H 7750 6000 50  0001 C CNN
+F 3 "" H 7750 6000 50  0001 C CNN
+	1    7750 6000
+	1    0    0    -1
+$EndComp
+Wire Wire Line
+	7150 5100 7750 5100
+Wire Wire Line
+	7750 5100 7750 6000
+Wire Wire Line
+	4700 5400 4700 5950
 $EndSCHEMATC

Commit message: v 1.1: Transistor footprint changed, resistor value changed
Parts:
- removed Q1: 2N3904, Package_TO_SOT_THT:TO-92_Inline, symbol Device:Q_NPN_BCE
- added Q1: 2N3904, Package_TO_SOT_THT:TO-92_Inline, symbol Transistor_BJT:2N3904
- R2: value 100K -> 10K
Changed lines of the file:
@@
 	5700 3200 5700 3300
 Wire Wire Line
-	5350 2800 5350 3300
-Wire Wire Line
 	5050 2600 4850 2600
-Wire Wire Line
-	6050 2400 5350 2400
-Wire Wire Line
-	5350 2400 5350 2150
 Wire Wire Line
 	5350 1850 5350 1650
@@
 P 4700 2600
 F 0 "R2" V 4493 2600 50  0000 C CNN
-F 1 "100K" V 4584 2600 50  0000 C CNN
+F 1 "10K" V 4584 2600 50  0000 C CNN
 F 2 "Resistor_THT:R_Axial_DIN0207_L6.3mm_D2.5mm_P7.62mm_Horizontal" V 4630 2600 50  0001 C CNN
 F 3 "~" H 4700 2600 50  0001 C CNN
@@
 F 3 "" H 5350 3300 50  0001 C CNN
 	1    5350 3300
-	1    0    0    -1
-$EndComp
-Connection ~ 5350 2400
-$Comp
-L Device:Q_NPN_BCE Q1
-U 1 1 5B6FC9ED
-P 5250 2600
-F 0 "Q1" H 5441 2646 50  0000 L CNN
-F 1 "2N3904" H 5441 2555 50  0000 L CNN
-F 2 "Package_TO_SOT_THT:TO-92_Inline" H 5450 2700 50  0001 C CNN
-F 3 "~" H 5250 2600 50  0001 C CNN
-	1    5250 2600
 	1    0    0    -1
 $EndComp
@@
 Connection ~ 7800 2400
 $Comp
-L power:GND #PWR?
+L power:GND #PWR0109
 U 1 1 5B71BD00
 P 4700 5950
-F 0 "#PWR?" H 4700 5700 50  0001 C CNN
+F 0 "#PWR0109" H 4700 5700 50  0001 C CNN
 F 1 "GND" H 4705 5777 50  0000 C CNN
 F 2 "" H 4700 5950 50  0001 C CNN
@@
 $EndComp
 $Comp
-L power:GND #PWR?
+L power:GND #PWR0110
 U 1 1 5B71BD46
 P 7750 6000
-F 0 "#PWR?" H 7750 5750 50  0001 C CNN
+F 0 "#PWR0110" H 7750 5750 50  0001 C CNN
 F 1 "GND" H 7755 5827 50  0000 C CNN
 F 2 "" H 7750 6000 50  0001 C CNN
@@
 Wire Wire Line
 	4700 5400 4700 5950
+$Comp
+L Transistor_BJT:2N3904 Q1
+U 1 1 5BC39C2B
+P 5250 2600
+F 0 "Q1" H 5441 2646 50  0000 L CNN
+F 1 "2N3904" H 5441 2555 50  0000 L CNN
+F 2 "Package_TO_SOT_THT:TO-92_Inline" H 5450 2525 50  0001 L CIN
+F 3 "https://www.fairchildsemi.com/datasheets/2N/2N3904.pdf" H 5250 2600 50  0001 L CNN
+	1    5250 2600
+	1    0    0    -1
+$EndComp
+Wire Wire Line
+	5350 2150 5350 2400
+Wire Wire Line
+	5350 2800 5350 3300
+Wire Wire Line
+	6050 2400 5350 2400
+Connection ~ 5350 2400
 $EndSCHEMATC
